Commit message: Add files via upload

File: arm_description/urdf/arm.xacro (robot description, xacro)
@@ -6,7 +6,7 @@
 <link name="base_link">
   <inertial>
-    <origin xyz="0.09186573896272435 0.1532477520366234 0.43778742695259654" rpy="0 0 0"/>
-    <mass value="1667.6422669621295"/>
-    <inertia ixx="124.966053" iyy="92.131981" izz="143.471825" ixy="4.544575" iyz="-2.412054" ixz="-0.087121"/>
+    <origin xyz="0.08975572850595205 0.0901367108721232 0.311840857838731" rpy="0 0 0"/>
+    <mass value="2627.615416556275"/>
+    <inertia ixx="304.849738" iyy="198.080618" izz="278.949801" ixy="3.936726" iyz="-38.694562" ixz="-1.300165"/>
   </inertial>
   <visual>
@@ -27,6 +27,6 @@
   <inertial>
     <origin xyz="2.637181544529188e-07 -2.7982934619474875e-07 0.17822374504581118" rpy="0 0 0"/>
-    <mass value="1.5059584614949872"/>
-    <inertia ixx="0.011173" iyy="0.013342" izz="0.0033" ixy="-0.0" iyz="0.0" ixz="0.0"/>
+    <mass value="1.6352579253607185"/>
+    <inertia ixx="0.012133" iyy="0.014488" izz="0.003583" ixy="-0.0" iyz="0.0" ixz="0.0"/>
   </inertial>
   <visual>
@@ -44,14 +44,14 @@
   </collision>
 </link>
-<link name="Forearm_V1_1">
+<link name="forearm_1">
   <inertial>
-    <origin xyz="0.0006800464679361934 -3.275052628051722e-07 0.1958085088828576" rpy="0 0 0"/>
-    <mass value="2.4095062985173903"/>
-    <inertia ixx="0.055448" iyy="0.057986" izz="0.004285" ixy="-0.0" iyz="-0.0" ixz="0.000321"/>
+    <origin xyz="0.0006800464679361934 -0.19580877978424263 -2.7638884736447267e-08" rpy="0 0 0"/>
+    <mass value="2.616383101925449"/>
+    <inertia ixx="0.060209" iyy="0.004653" izz="0.062965" ixy="-0.000348" iyz="0.0" ixz="-0.0"/>
   </inertial>
   <visual>
     <origin xyz="-0.07609 0.044498 -0.976099" rpy="0 0 0"/>
     <geometry>
-      <mesh filename="package://arm_description/meshes/Forearm_V1_1.stl" scale="0.001 0.001 0.001"/>
+      <mesh filename="package://arm_description/meshes/forearm_1.stl" scale="0.001 0.001 0.001"/>
     </geometry>
     <material name="silver"/>
@@ -60,5 +60,5 @@
     <origin xyz="-0.07609 0.044498 -0.976099" rpy="0 0 0"/>
     <geometry>
-      <mesh filename="package://arm_description/meshes/Forearm_V1_1.stl" scale="0.001 0.001 0.001"/>
+      <mesh filename="package://arm_description/meshes/forearm_1.stl" scale="0.001 0.001 0.001"/>
     </geometry>
   </collision>
@@ -66,10 +66,10 @@
 <link name="hand_1">
   <inertial>
-    <origin xyz="0.0020797334823772495 -3.2885904838186875e-07 0.09682033280236535" rpy="0 0 0"/>
-    <mass value="1.5143538846168256"/>
-    <inertia ixx="0.016077" iyy="0.016569" izz="0.001364" ixy="-0.0" iyz="0.0" ixz="0.000305"/>
+    <origin xyz="0.0020797334823772357 -0.09682060370375017 -2.899267115274995e-08" rpy="0 0 0"/>
+    <mass value="1.6443741676394823"/>
+    <inertia ixx="0.017457" iyy="0.001481" izz="0.017991" ixy="-0.000331" iyz="-0.0" ixz="-0.0"/>
   </inertial>
   <visual>
-    <origin xyz="-0.07609 0.044498 -1.376099" rpy="0 0 0"/>
+    <origin xyz="-0.07609 0.444498 -0.976099" rpy="0 0 0"/>
     <geometry>
       <mesh filename="package://arm_description/meshes/hand_1.stl" scale="0.001 0.001 0.001"/>
@@ -78,5 +78,5 @@
   </visual>
   <collision>
-    <origin xyz="-0.07609 0.044498 -1.376099" rpy="0 0 0"/>
+    <origin xyz="-0.07609 0.444498 -0.976099" rpy="0 0 0"/>
     <geometry>
       <mesh filename="package://arm_description/meshes/hand_1.stl" scale="0.001 0.001 0.001"/>
@@ -86,10 +86,10 @@
 <link name="fork_1">
   <inertial>
-    <origin xyz="2.639346036725776e-07 -3.185903194521944e-07 0.06732396455714396" rpy="0 0 0"/>
-    <mass value="0.920458057868743"/>
-    <inertia ixx="0.001655" iyy="0.003944" izz="0.003257" ixy="0.0" iyz="0.0" ixz="0.0"/>
+    <origin xyz="2.639346036725776e-07 -0.06732423545852861 -1.8723942840637164e-08" rpy="0 0 0"/>
+    <mass value="0.9994872850594936"/>
+    <inertia ixx="0.001797" iyy="0.003536" izz="0.004282" ixy="-0.0" iyz="-0.0" ixz="0.0"/>
   </inertial>
   <visual>
-    <origin xyz="-0.07609 0.044498 -1.666099" rpy="0 0 0"/>
+    <origin xyz="-0.07609 0.734498 -0.976099" rpy="0 0 0"/>
     <geometry>
       <mesh filename="package://arm_description/meshes/fork_1.stl" scale="0.001 0.001 0.001"/>
@@ -98,5 +98,5 @@
   </visual>
   <collision>
-    <origin xyz="-0.07609 0.044498 -1.666099" rpy="0 0 0"/>
+    <origin xyz="-0.07609 0.734498 -0.976099" rpy="0 0 0"/>
     <geometry>
       <mesh filename="package://arm_description/meshes/fork_1.stl" scale="0.001 0.001 0.001"/>
@@ -104,21 +104,21 @@
   </collision>
 </link>
-<link name="end_effector__1__1">
+<link name="end_effector_1">
   <inertial>
-    <origin xyz="0.04687257576486922 -3.14966209571943e-07 0.05916220318041665" rpy="0 0 0"/>
-    <mass value="1.006827933659346"/>
-    <inertia ixx="0.008518" iyy="0.009009" izz="0.001046" ixy="-0.0" iyz="0.0" ixz="-0.000186"/>
+    <origin xyz="0.046872575764868515 -0.05916247408180153 -1.5099832273435254e-08" rpy="0 0 0"/>
+    <mass value="1.0932727562462594"/>
+    <inertia ixx="0.009249" iyy="0.001136" izz="0.009782" ixy="0.000202" iyz="-0.0" ixz="-0.0"/>
   </inertial>
   <visual>
-    <origin xyz="-0.02609 0.044498 -1.776099" rpy="0 0 0"/>
+    <origin xyz="-0.02609 0.844498 -0.976099" rpy="0 0 0"/>
     <geometry>
-      <mesh filename="package://arm_description/meshes/end_effector__1__1.stl" scale="0.001 0.001 0.001"/>
+      <mesh filename="package://arm_description/meshes/end_effector_1.stl" scale="0.001 0.001 0.001"/>
     </geometry>
     <material name="silver"/>
   </visual>
   <collision>
-    <origin xyz="-0.02609 0.044498 -1.776099" rpy="0 0 0"/>
+    <origin xyz="-0.02609 0.844498 -0.976099" rpy="0 0 0"/>
     <geometry>
-      <mesh filename="package://arm_description/meshes/end_effector__1__1.stl" scale="0.001 0.001 0.001"/>
+      <mesh filename="package://arm_description/meshes/end_effector_1.stl" scale="0.001 0.001 0.001"/>
     </geometry>
   </collision>
@@ -130,27 +130,30 @@
   <axis xyz="0.0 0.0 1.0"/>
 </joint>
-<joint name="joint_2" type="continuous">
+<joint name="joint_2" type="revolute">
   <origin xyz="0.0 0.0 0.28" rpy="0 0 0"/>
   <parent link="shoulder_1"/>
-  <child link="Forearm_V1_1"/>
+  <child link="forearm_1"/>
   <axis xyz="1.0 0.0 -0.0"/>
+  <limit upper="0.349066" lower="-3.490659" effort="100" velocity="100"/>
 </joint>
-<joint name="joint_3" type="continuous">
-  <origin xyz="0.0 0.0 0.4" rpy="0 0 0"/>
-  <parent link="Forearm_V1_1"/>
+<joint name="joint_3" type="revolute">
+  <origin xyz="0.0 -0.4 0.0" rpy="0 0 0"/>
+  <parent link="forearm_1"/>
   <child link="hand_1"/>
-  <axis xyz="1.0 -0.0 -0.0"/>
+  <axis xyz="1.0 0.0 -0.0"/>
+  <limit upper="1.919862" lower="-1.919862" effort="100" velocity="100"/>
 </joint>
 <joint name="joint_4" type="continuous">
-  <origin xyz="0.0 0.0 0.29" rpy="0 0 0"/>
+  <origin xyz="0.0 -0.29 0.0" rpy="0 0 0"/>
   <parent link="hand_1"/>
   <child link="fork_1"/>
-  <axis xyz="-0.0 0.0 -1.0"/>
+  <axis xyz="0.0 1.0 0.0"/>
 </joint>
-<joint name="joint_5" type="continuous">
-  <origin xyz="-0.05 0.0 0.11" rpy="0 0 0"/>
+<joint name="joint_5" type="revolute">
+  <origin xyz="-0.05 -0.11 0.0" rpy="0 0 0"/>
   <parent link="fork_1"/>
-  <child link="end_effector__1__1"/>
-  <axis xyz="1.0 -0.0 0.0"/>
+  <child link="end_effector_1"/>
+  <axis xyz="1.0 0.0 -0.0"/>
+  <limit upper="2.094395" lower="-2.094395" effort="100" velocity="100"/>
 </joint>
 </robot>
